Commit message: 坐标位置正确

File: src/BRX042501/urdf/BRX042501_fixed_wheel_change_axis.urdf (robot description, URDF)
Before this commit: robot BRX042501, 45 links, 44 joints
Links:
- added link base_dummy
Joints:
- added joint fixed_base_joint: type fixed, parent base_dummy, child base_link, origin xyz=0 0 0 rpy=0 0 0
